Commit message: Change kinect orientation

File: drake/examples/kuka_iiwa_arm/models/objects/xtion.urdf (robot description, URDF)
Before this commit: robot xtion, 2 links, 1 joints
Links:
- added link xtion_base
Joints:
- added joint xtion_base: type fixed, parent xtion_base, child xtion, origin xyz=0 0 0 rpy=1.57 0 1.57
- joint xtion_to_lens: origin xyz=0.0 0 0.0 rpy=0 0 0 -> xyz=0.0 0 0.0 rpy=0 0.0 0
