Commit message: tree tester fixed

File: drake/examples/kuka_iiwa_arm/models/objects/book.urdf (robot description, URDF)
Before this commit: robot book, 1 links, 0 joints
Links:
- link base_link: mass 0.68 -> 0.50; geometry collision box size=0.229 0.179 0.009; collision sphere radius=1e-7

Commit message: Needs tuning

File: drake/examples/kuka_iiwa_arm/models/objects/book.urdf (robot description, URDF)
Before this commit: robot book, 1 links, 0 joints
Links:
- link base_link: geometry collision box size=0.229 0.179 0.009; collision sphere radius=1e-7
