Commit message: Add decimated meshes

File: drake/manipulation/models/iiwa_description/urdf/iiwa14.xacro (robot description, xacro)
@@ -14,5 +14,5 @@
   <xacro:property name="max_velocity" value="10"/>
   <xacro:macro name="iiwa14"
-      params="parent hardware_interface robot_name collision_type *origin">
+      params="parent hardware_interface robot_name collision_type *origin mesh_collision_directory:=meshes/collision">
     <!--joint between {parent} and link_0-->
     <joint name="${robot_name}_${parent}_joint" type="fixed">
@@ -38,5 +38,5 @@
           <origin xyz="0 0 0" rpy="0 0 0"/>
           <geometry>
-            <mesh filename="../meshes/collision/link_0.obj"/>
+            <mesh filename="../${mesh_collision_directory}/link_0.obj"/>
           </geometry>
           <material name="Grey"/>
@@ -91,5 +91,5 @@
           <origin xyz="0 0 0" rpy="0 0 0"/>
           <geometry>
-            <mesh filename="../meshes/collision/link_1.obj"/>
+            <mesh filename="../${mesh_collision_directory}/link_1.obj"/>
           </geometry>
           <material name="Grey"/>
@@ -138,5 +138,5 @@
           <origin xyz="0 0 0" rpy="0 0 0"/>
           <geometry>
-            <mesh filename="../meshes/collision/link_2.obj"/>
+            <mesh filename="../${mesh_collision_directory}/link_2.obj"/>
           </geometry>
           <material name="Orange"/>
@@ -185,5 +185,5 @@
           <origin xyz="0 0 0" rpy="0 0 0"/>
           <geometry>
-            <mesh filename="../meshes/collision/link_3.obj"/>
+            <mesh filename="../${mesh_collision_directory}/link_3.obj"/>
           </geometry>
           <material name="Grey"/>
@@ -232,5 +232,5 @@
           <origin xyz="0 0 0" rpy="0 0 0"/>
           <geometry>
-            <mesh filename="../meshes/collision/link_4.obj"/>
+            <mesh filename="../${mesh_collision_directory}/link_4.obj"/>
           </geometry>
           <material name="Orange"/>
@@ -279,5 +279,5 @@
           <origin xyz="0 0 0" rpy="0 0 0"/>
           <geometry>
-            <mesh filename="../meshes/collision/link_5.obj"/>
+            <mesh filename="../${mesh_collision_directory}/link_5.obj"/>
           </geometry>
           <material name="Grey"/>
@@ -326,5 +326,5 @@
           <origin xyz="0 0 0" rpy="0 0 0"/>
           <geometry>
-            <mesh filename="../meshes/collision/link_6.obj"/>
+            <mesh filename="../${mesh_collision_directory}/link_6.obj"/>
           </geometry>
           <material name="Orange"/>
@@ -337,5 +337,5 @@
             <!-- Note that the mesh-based collision model is intentionally being
             used despite being in "primitive" mode. -->
-            <mesh filename="../meshes/collision/link_6.obj"/>
+            <mesh filename="../${mesh_collision_directory}/link_6.obj"/>
           </geometry>
           <material name="Orange"/>
@@ -375,5 +375,5 @@
           <origin xyz="0 0 0" rpy="0 0 0"/>
           <geometry>
-            <mesh filename="../meshes/collision/link_7.obj"/>
+            <mesh filename="../${mesh_collision_directory}/link_7.obj"/>
           </geometry>
           <material name="Grey"/>
@@ -386,5 +386,5 @@
             <!-- Note that the mesh-based collision model is intentionally being
             used despite being in "primitive" mode. -->
-            <mesh filename="../meshes/collision/link_7.obj"/>
+            <mesh filename="../${mesh_collision_directory}/link_7.obj"/>
           </geometry>
           <material name="Grey"/>
@@ -395,5 +395,5 @@
           <origin xyz="0 0 0" rpy="0 0 0"/>
           <geometry>
-            <mesh filename="../meshes/collision/link_7_polytope.obj"/>
+            <mesh filename="../${mesh_collision_directory}/link_7_polytope.obj"/>
           </geometry>
           <material name="Grey"/>
