Commit message: Make Python fail

File: tmp/hamr_scaled.urdf (robot description, URDF)
Before this commit: robot Hamr, 33 links, 32 joints
Links:
- link Chassis: geometry 
- link FLL1: geometry 
- link FLL2: geometry 
- link FLL3: geometry 
- link FLL4: geometry collision sphere radius=0
- link FLS1: geometry 
- link FLS2: geometry 
- link FLS3: geometry 
- link FLS4: geometry 
- link FRL1: geometry 
- link FRL2: geometry 
- link FRL3: geometry 
- link FRL4: geometry collision sphere radius=0
- link FRS1: geometry 
- link FRS2: geometry 
- link FRS3: geometry 
- link FRS4: geometry 
- link RLL1: geometry 
- link RLL2: geometry 
- link RLL3: geometry 
- link RLL4: geometry collision sphere radius=0
- link RLS1: geometry 
- link RLS2: geometry 
- link RLS3: geometry 
- link RLS4: geometry 
- link RRL1: geometry 
- link RRL2: geometry 
- link RRL3: geometry 
- link RRL4: geometry collision sphere radius=0
- link RRS1: geometry 
- link RRS2: geometry 
- link RRS3: geometry 
- link RRS4: geometry 

Commit message: Smaller repro

File: tmp/hamr_scaled.urdf (robot description, URDF)
Before this commit: robot Hamr, 33 links, 32 joints
Links:
- link Chassis: geometry visual sphere radius=0.05
- link FLL1: geometry visual sphere radius=0.05
- link FLL2: geometry visual sphere radius=0.05
- link FLL3: geometry visual sphere radius=0.05
- link FLL4: geometry collision sphere radius=0; visual sphere radius=0.05
- link FLS1: geometry visual sphere radius=0.05
- link FLS2: geometry visual sphere radius=0.05
- link FLS3: geometry visual sphere radius=0.05
- link FLS4: geometry visual sphere radius=0.05
- link FRL1: geometry visual sphere radius=0.05
- link FRL2: geometry visual sphere radius=0.05
- link FRL3: geometry visual sphere radius=0.05
- link FRL4: geometry collision sphere radius=0; visual sphere radius=0.05
- link FRS1: geometry visual sphere radius=0.05
- link FRS2: geometry visual sphere radius=0.05
- link FRS3: geometry visual sphere radius=0.05
- link FRS4: geometry visual sphere radius=0.05
- link RLL1: geometry visual sphere radius=0.05
- link RLL2: geometry visual sphere radius=0.05
- link RLL3: geometry visual sphere radius=0.05
- link RLL4: geometry collision sphere radius=0; visual sphere radius=0.05
- link RLS1: geometry visual sphere radius=0.05
- link RLS2: geometry visual sphere radius=0.05
- link RLS3: geometry visual sphere radius=0.05
- link RLS4: geometry visual sphere radius=0.05
- link RRL1: geometry visual sphere radius=0.05
- link RRL2: geometry visual sphere radius=0.05
- link RRL3: geometry visual sphere radius=0.05
- link RRL4: geometry collision sphere radius=0; visual sphere radius=0.05
- link RRS1: geometry visual sphere radius=0.05
- link RRS2: geometry visual sphere radius=0.05
- link RRS3: geometry visual sphere radius=0.05
- link RRS4: geometry visual sphere radius=0.05
